File: 514final/514final.kicad_pcb (KiCad board)
At the start: 2 copper layers, 2 parts

Commit message: v3.0
Parts:
- removed S1: B3F-1000, B3F-1000:SW_B3F-1000
- added BT1: Battery_Cell, Connector_JST:JST_NV_B02P-NV_1x02_P5.00mm_Vertical, F.Cu at (184.2, 141.0)
- added D1: LED_RGBK, LED_THT:LED_D5.0mm-4_RGB_Staggered_Pins, F.Cu at (189.2, 108.0)
- added M1: Stepper_Motor_bipolar, x27_Footprint:x27_stepper, B.Cu at (203.2, 132.1)
- added R1: R, Resistor_SMD:R_0805_2012Metric_Pad1.20x1.40mm_HandSolder, F.Cu at (221.2, 108.0)
- added R2: R, Resistor_SMD:R_0805_2012Metric_Pad1.20x1.40mm_HandSolder, F.Cu at (211.1, 97.8)
- added R3: R, Resistor_SMD:R_0805_2012Metric_Pad1.20x1.40mm_HandSolder, F.Cu at (216.2, 102.9)
- added SW1: SW_SPDT, Connector_JST:JST_EH_B3B-EH-A_1x03_P2.50mm_Vertical, F.Cu at (237.5, 141.0)
- U1: moved to B.Cu
- moved U1 192.1 mm to (241.3, 116.8), turned to 90 degrees
Connections:
- U1 pad 1: unconnected-(U1-GPIO1_A0_D0-Pad1) -> Net-(U1-GPIO1_A0_D0)
- U1 pad 11: unconnected-(U1-GPIO9_A10_D10_COPI-Pad11) -> Net-(U1-GPIO9_A10_D10_COPI)
- U1 pad 12: unconnected-(U1-GPIO8_A9_D9_CIPO-Pad12) -> Net-(U1-GPIO8_A9_D9_CIPO)
- U1 pad 13: unconnected-(U1-GPIO7_A8_D8_SCK-Pad13) -> Net-(U1-GPIO7_A8_D8_SCK)
- U1 pad 2: unconnected-(U1-GPIO2_A1_D1-Pad2) -> Net-(M1--)
- U1 pad 3: unconnected-(U1-GPIO3_A2_D2-Pad3) -> Net-(U1-GPIO3_A2_D2)
- U1 pad 4: unconnected-(U1-GPIO4_A3_D3-Pad4) -> Net-(U1-GPIO4_A3_D3)
- U1 pad 8: unconnected-(U1-5V-Pad8) -> Net-(SW1-C)
- U1 pad 9: unconnected-(U1-GND-Pad9) -> Net-(BT1--)
Routing:
- net Net-(BT1--): track 0.00 -> 103.5 mm
- net Net-(U1-GPIO1_A0_D0): track 0.00 -> 64.9 mm
- net Net-(M1--): track 0.00 -> 61.9 mm
- net Net-(BT1-+): track 0.00 -> 57.0 mm
- net Net-(SW1-C): track 0.00 -> 35.6 mm
- net Net-(D1-BA): track 0.00 -> 35.4 mm
- net Net-(U1-GPIO9_A10_D10_COPI): track 0.00 -> 34.5 mm
- net Net-(U1-GPIO3_A2_D2): track 0.00 -> 31.8 mm
- net Net-(D1-RA): track 0.00 -> 28.0 mm
- net Net-(U1-GPIO4_A3_D3): track 0.00 -> 26.8 mm
- net Net-(D1-GA): track 0.00 -> 26.2 mm
- net Net-(U1-GPIO7_A8_D8_SCK): track 0.00 -> 22.2 mm
- net Net-(U1-GPIO8_A9_D9_CIPO): track 0.00 -> 18.2 mm
Other:
- board outline added: 78.7 x 53.3 mm
- board text added: "Ruiqing Wang Display PCB V3.0"
