File: 514final/514final.kicad_sch (KiCad schematic)
At the start: 2 parts

Commit message: v3.0
Parts:
- removed S1: B3F-1000, B3F-1000:SW_B3F-1000, symbol button:B3F-1000
- added BT1: Battery_Cell, Connector_JST:JST_NV_B02P-NV_1x02_P5.00mm_Vertical, symbol Device:Battery_Cell
- added D1: LED_RGBK, LED_THT:LED_D5.0mm-4_RGB_Staggered_Pins, symbol Device:LED_RGBK
- added M1: Stepper_Motor_bipolar, x27_Footprint:x27_stepper, symbol Motor:Stepper_Motor_bipolar
- added R1, R2, R3: R, Resistor_SMD:R_0805_2012Metric_Pad1.20x1.40mm_HandSolder, symbol Device:R
- added SW1: SW_SPDT, Connector_JST:JST_EH_B3B-EH-A_1x03_P2.50mm_Vertical, symbol Switch:SW_SPDT
Connections:
- net at U1.1 (GPIO1_A0_D0): now also M1.1
- net at U1.11 (GPIO9_A10_D10_COPI): now also R2.2
- net at U1.12 (GPIO8_A9_D9_CIPO): now also R1.2
- net at U1.13 (GPIO7_A8_D8_SCK): now also R3.2
- net at U1.2 (GPIO2_A1_D1): now also M1.2 (-)
- net at U1.3 (GPIO3_A2_D2): now also M1.3
- net at U1.4 (GPIO4_A3_D3): now also M1.4
- net at U1.8 (5V): now also SW1.3 (C)
- net at U1.9 (GND): now also BT1.2 (-), D1.4 (K)
- new net: D1.1 (RA), R3.1
- new net: D1.3 (BA), R1.1
- new net: BT1.1 (+), SW1.2 (B)
- new net: D1.2 (GA), R2.1
Other:
- title: (none) -> Ruiqing Wang's Display PCB V2.0
- moved on the sheet: U1
